File: mcu_datalogger.kicad_sch (KiCad schematic)
At the start: 0 parts

Commit message: Schematic update
Parts:
- added BT1: Battery, symbol Device:Battery
- added C1, C2, C3, C4: C, symbol Device:C
- added C5: C_Polarized, symbol Device:C_Polarized
- added D1, D2: LED, symbol Device:LED
- added H1, H2, H3, H4: MountingHole, symbol Mechanical:MountingHole
- added R1, R2, R3, R4, R5, R6, R7: R, symbol Device:R
- added U1, U2: 24LC1025, Package_DFN_QFN:WDFN-8-1EP_6x5mm_P1.27mm_EP3.4x4mm, symbol Memory_EEPROM:24LC1025
- added U3: DS1337S_, DS1337S_:SOIC127P600X175-8N, symbol DS1337S_:DS1337S_
- added U4: ATMEGA328P-AU_SL044, ATMEGA328P-AU_SL044:QFP80P900X900X120-32N, symbol ATMEGA328P-AU_SL044:ATMEGA328P-AU_SL044
- added Y1, Y2: Crystal, symbol Device:Crystal
Connections:
- new net GND: U4.21 (GND), U4.3 (GND), U4.5 (GND)
- new net VCC: U4.4 (VCC), U4.6 (VCC)
Other:
- added sheet Connectors (connectors.kicad_sch)
- title: (none) -> ${project_name}

Commit message: Schematic update v2
Parts:
- C1, C4: value C -> 0.1uF
- C2, C3: value C -> 22uF
- C5: value C_Polarized -> 100nF
- R1, R2, R6: value R -> 10K
- R3, R4: value R -> 4.7K
- R5, R7: value R -> 330
- Y1: value Crystal -> 32.768 KHz
- Y2: value Crystal -> 16 MHz
- renumbered U3 to U2, U2 to U3
Other:
- moved on the sheet: BT1, C1, C2, C3, C4, C5, D1, D2, H1, H2, H3, H4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

Commit message: Schematic update v3
Parts:
- BT1: footprint (none) -> Connector_PinHeader_2.54mm:PinHeader_1x02_P2.54mm_Vertical
- C1, C2, C3, C4, C5: footprint (none) -> Capacitor_SMD:C_0805_2012Metric
- D1, D2: footprint (none) -> LED_SMD:LED_0805_2012Metric
- H1, H2, H3, H4: footprint (none) -> MountingHole:MountingHole_2.1mm
- R1, R2, R3, R4, R5, R6, R7: footprint (none) -> Resistor_SMD:R_0805_2012Metric
- U1, U3: footprint Package_DFN_QFN:WDFN-8-1EP_6x5mm_P1.27mm_EP3.4x4mm -> Package_SO:SOIC-8_5.23x5.23mm_P1.27mm
- Y1, Y2: footprint (none) -> Crystal:Crystal_SMD_5032-2Pin_5.0x3.2mm_HandSoldering
Connections:
- net GND: now also BT1.2 (-), C1.1, C5.2, R7.1, U1.4 (GND), U1.7 (WP), U2.4 (GND), U3.2 (A1), U3.4 (GND), U3.7 (WP)
- net Vcc: now reaches U3.1 (A0)
- net Vcc: now also C1.2, R1.1, R2.2, R3.1, R4.1, R6.1, U1.1 (A0), U1.2 (A1), U1.3 (A2), U1.8 (VCC), U2.8 (VCC), U3.3 (A2), U3.8 (VCC)
- net SDA: now reaches U3.5 (SDA)
- net SDA: now also R4.2, U1.5 (SDA), U2.5 (SDA)
- net SCK: now reaches U3.6 (SCL)
- net SCK: now also R3.2, U1.6 (SCL), U2.6 (SCL)
- net at U2.1 (X1): now also Y1.2
- net at U2.2 (X2): now also Y1.1
- net at U2.3 (~{INTA}): now also R1.2
- net at U2.7 (SQW/~INT): now also R2.1
- net at R7.2: now also D2.1 (K)
- net at D2.2 (A): now also BT1.1 (+), C5.1, U4.18 (AVCC)
- net at R6.2: now also U4.29 (PC6/~{RESET})
- net at U4.7 (PB6): now also Y2.2
- net at U4.8 (PB7): now also Y2.1
- net VCC: no longer names the net of U4.4 (VCC)
- net VCC: no longer U4.6 (VCC)
Other:
- note added: "CLOCK"
- moved on the sheet: BT1, C5, D2, R3, R4, R6, R7, U1, U3, Y1, Y2

Commit message: Schematic update final
Connections:
- net GND: now also C2.2, C3.2, C4.1, R5.1
- net SCK: now also D1.2 (A), U4.17 (PB5), U4.28 (PC5)
- net SDA: now also U4.27 (PC4)
- net at C2.1: now also U4.7 (PB6), Y2.2
- net at D1.1 (K): now also R5.2
- net at BT1.1 (+), C5.1, D2.2 (A)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: now also U4.4 (VCC)
- net at C3.1: now also U4.8 (PB7), Y2.1
- net RESET: now reaches R6.2, U4.29 (PC6/~{RESET})
- net D3: now reaches U4.1 (PD3)
- net D6: now reaches U4.10 (PD6)
- net D7: now reaches U4.11 (PD7)
- net D8: now reaches U4.12 (PB0)
- net MOSI: now reaches U4.15 (PB3)
- net MISO: now reaches U4.16 (PB4)
- net D4: now reaches U4.2 (PD4)
- net at U4.20 (AREF): now also C4.2
- net RX: now reaches U4.30 (PD0)
- net TX: now reaches U4.31 (PD1)
- net D2: now reaches U4.32 (PD2)
- net D5: now reaches U4.9 (PD5)
- no-connect marks 0 -> 9
Other:
- sheet Connectors ports: added D2, D3, D4, D5, D6, D7, D8, GND, MISO, MOSI, RESET, RX, SCK, SDA, TX, Vcc; removed none
- note added: "EEPROM"
- note added: "MICROCONTROLLER UNIT"
- note added: "MOUNTING HOLES"
- note added: "REAL TIME CLOCK"
- note removed: "CLOCK"
- moved on the sheet: C2, C3, C4, Y2

Commit message: PCB - small fix
Other:
- note removed: "MOUNTING HOLES"
Changed lines of the file:
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@@
-	)
-	(rectangle
-		(start 242.57 127.508)
-		(end 271.272 154.94)
-		(stroke
-			(width 0)
-			(type default)
-		)
-		(fill
-			(type none)
-		)
 	)
 	(rectangle
@@
 		)
 	)
-	(text "MOUNTING HOLES"
-		(exclude_from_sim no)
-		(at 250.19 126.365 0)
-		(effects
-			(font
-				(size 1.27 1.27)
-			)
-		)
-	)

Commit message: Finished
Connections:
- net Vcc: now also BT1.1 (+), C5.1, D2.2 (A), U4.18 (AVCC), U4.4 (VCC)
Changed lines of the file:
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@@
+		)
+	)
+	(label "Vcc"
+		(at 234.315 38.1 0)
+		(effects
+			(font
+				(size 1.27 1.27)
+			)
+			(justify left bottom)
 		)
 	)

Commit message: bugfix
Connections:
- net SCK: no longer U1.6 (SCL), U2.6 (SCL), U3.6 (SCL), U4.28 (PC5)
- new net SCL: U1.6 (SCL), U2.6 (SCL), U3.6 (SCL), U4.28 (PC5)
Other:
- sheet Connectors ports: added SCL; removed none
Changed lines of the file:
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@@
 	(wire
 		(pts
-			(xy 226.06 29.21) (xy 226.06 38.1)
-		)
-		(stroke
-			(width 0)
-			(type default)
-		)
-	)
-	(wire
-		(pts
 			(xy 64.77 154.94) (xy 73.66 154.94)
 		)
@@
 		)
 	)
-	(label "SCK"
+	(label "SCL"
 		(at 185.42 81.28 180)
 		(effects
@@
 		)
 	)
-	(label "SCK"
+	(label "SCL"
 		(at 171.45 132.08 180)
 		(effects
@@
 		)
 	)
-	(label "SCK"
+	(label "SCL"
 		(at 45.72 48.26 180)
 		(effects
@@
 		)
 	)
-	(label "SCK"
+	(label "SCL"
 		(at 100.33 147.32 0)
 		(effects
@@
 		)
 	)
+	(label "SCK"
+		(at 171.45 141.605 180)
+		(effects
+			(font
+				(size 1.27 1.27)
+			)
+			(justify right bottom)
+		)
+	)
 	(label "SDA"
 		(at 64.77 144.78 0)
@@
 		)
 	)
-	(label "SCK"
+	(label "SCL"
 		(at 64.77 147.32 0)
 		(effects
@@
 	)
 	(label "RESET"
-		(at 171.45 147.32 180)
+		(at 171.45 149.225 180)
 		(effects
 			(font
@@
 	)
 	(label "MISO"
-		(at 171.45 144.78 180)
+		(at 171.45 146.685 180)
 		(effects
 			(font
@@
 	)
 	(label "MOSI"
-		(at 171.45 142.24 180)
+		(at 171.45 144.145 180)
 		(effects
 			(font
@@
 	)
 	(symbol
-		(lib_id "power:PWR_FLAG")
-		(at 226.06 29.21 0)
-		(unit 1)
-		(body_style 1)
-		(exclude_from_sim no)
-		(in_bom yes)
-		(on_board yes)
-		(in_pos_files yes)
-		(dnp no)
-		(fields_autoplaced yes)
-		(property "Reference" "#FLG01"
-			(at 226.06 27.305 0)
-			(hide yes)
-			(show_name no)
-			(do_not_autoplace no)
-			(effects
-				(font
-					(size 1.27 1.27)
-				)
-			)
-		)
-		(property "Value" "PWR_FLAG"
-			(at 226.06 24.13 0)
-			(show_name no)
-			(do_not_autoplace no)
-			(effects
-				(font
-					(size 1.27 1.27)
-				)
-			)
-		)
-		(property "Footprint" "Package_SO:TSSOP-28_4.4x9.7mm_P0.65mm"
-			(at 226.06 29.21 0)
-			(hide yes)
-			(show_name no)
-			(do_not_autoplace no)
-			(effects
-				(font
-					(size 1.27 1.27)
-				)
-			)
-		)
-		(property "Datasheet" ""
-			(at 226.06 29.21 0)
-			(hide yes)
-			(show_name no)
-			(do_not_autoplace no)
-			(effects
-				(font
-					(size 1.27 1.27)
-				)
-			)
-		)
-		(property "Description" "Special symbol for telling ERC where power comes from"
-			(at 226.06 29.21 0)
-			(hide yes)
-			(show_name no)
-			(do_not_autoplace no)
-			(effects
-				(font
-					(size 1.27 1.27)
-				)
-			)
-		)
-		(pin "1"
-		)
-		(instances
-			(project "mcu_datalogger"
-				(path "/c956c193-eb19-4c5d-8ea2-20354ad9de1d"
-					(reference "#FLG01")
-					(unit 1)
-				)
-			)
-		)
-	)
-	(symbol
 		(lib_id "Device:R")
 		(at 146.05 48.26 90)
@@
 		)
 		(pin "MOSI" input
-			(at 171.45 142.24 180)
+			(at 171.45 144.145 180)
 			(effects
 				(font
@@
 		)
 		(pin "RESET" passive
-			(at 171.45 147.32 180)
+			(at 171.45 149.225 180)
 			(effects
 				(font
@@
 		)
 		(pin "MISO" output
-			(at 171.45 144.78 180)
+			(at 171.45 146.685 180)
 			(effects
 				(font
@@
 			)
 		)
-		(pin "SCK" passive
+		(pin "SCL" passive
 			(at 171.45 132.08 180)
 			(effects
 				(font
+					(size 1.27 1.27)
+				)
+				(justify left)
+			)
+		)
+		(pin "SCK" passive
+			(at 171.45 141.605 180)
+			(effects
+				(font
