File: mcu_datalogger.kicad_sch (KiCad schematic)
At the start: 25 parts, among them U1 24LC1025, U2 DS1337S_, U3 24LC1025, U4 ATMEGA328P-AU_SL044, Y1 32.768 KHz, Y2 16 MHz

Commit message: bugfix
Connections:
- net SCK: no longer U1.6 (SCL), U2.6 (SCL), U3.6 (SCL), U4.28 (PC5)
- net Vcc: now also BT1.1 (+), C5.1, D2.2 (A), U4.18 (AVCC), U4.4 (VCC)
- new net SCL: U1.6 (SCL), U2.6 (SCL), U3.6 (SCL), U4.28 (PC5)
Other:
- sheet Connectors ports: added SCL; removed none
- note removed: "MOUNTING HOLES"
Changed lines of the file:
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@@
 	)
 	(rectangle
-		(start 242.57 127.508)
-		(end 271.272 154.94)
-		(stroke
-			(width 0)
-			(type default)
-		)
-		(fill
-			(type none)
-		)
-	)
-	(rectangle
 		(start 132.715 19.685)
 		(end 259.08 104.14)
@@
 		)
 	)
-	(text "MOUNTING HOLES"
-		(exclude_from_sim no)
-		(at 250.19 126.365 0)
-		(effects
-			(font
-				(size 1.27 1.27)
-			)
-		)
-	)
 	(text "MICROCONTROLLER UNIT"
 		(exclude_from_sim no)
@@
 	(wire
 		(pts
-			(xy 226.06 29.21) (xy 226.06 38.1)
-		)
-		(stroke
-			(width 0)
-			(type default)
-		)
-	)
-	(wire
-		(pts
 			(xy 64.77 154.94) (xy 73.66 154.94)
 		)
@@
 		)
 	)
-	(label "SCK"
+	(label "SCL"
 		(at 185.42 81.28 180)
 		(effects
@@
 		)
 	)
-	(label "SCK"
+	(label "SCL"
 		(at 171.45 132.08 180)
 		(effects
@@
 		)
 	)
-	(label "SCK"
+	(label "SCL"
 		(at 45.72 48.26 180)
 		(effects
@@
 		)
 	)
-	(label "SCK"
+	(label "SCL"
 		(at 100.33 147.32 0)
 		(effects
@@
 		)
 	)
+	(label "SCK"
+		(at 171.45 141.605 180)
+		(effects
+			(font
+				(size 1.27 1.27)
+			)
+			(justify right bottom)
+		)
+	)
 	(label "SDA"
 		(at 64.77 144.78 0)
@@
 		)
 	)
-	(label "SCK"
+	(label "SCL"
 		(at 64.77 147.32 0)
 		(effects
@@
 	)
 	(label "RESET"
-		(at 171.45 147.32 180)
+		(at 171.45 149.225 180)
 		(effects
 			(font
@@
 	)
 	(label "MISO"
-		(at 171.45 144.78 180)
+		(at 171.45 146.685 180)
 		(effects
 			(font
@@
 	)
 	(label "MOSI"
-		(at 171.45 142.24 180)
+		(at 171.45 144.145 180)
 		(effects
 			(font
@@
 		)
 	)
+	(label "Vcc"
+		(at 234.315 38.1 0)
+		(effects
+			(font
+				(size 1.27 1.27)
+			)
+			(justify left bottom)
+		)
+	)
 	(label "SCK"
 		(at 185.42 58.42 180)
@@
 	)
 	(symbol
-		(lib_id "power:PWR_FLAG")
-		(at 226.06 29.21 0)
-		(unit 1)
-		(body_style 1)
-		(exclude_from_sim no)
-		(in_bom yes)
-		(on_board yes)
-		(in_pos_files yes)
-		(dnp no)
-		(fields_autoplaced yes)
-		(property "Reference" "#FLG01"
-			(at 226.06 27.305 0)
-			(hide yes)
-			(show_name no)
-			(do_not_autoplace no)
-			(effects
-				(font
-					(size 1.27 1.27)
-				)
-			)
-		)
-		(property "Value" "PWR_FLAG"
-			(at 226.06 24.13 0)
-			(show_name no)
-			(do_not_autoplace no)
-			(effects
-				(font
-					(size 1.27 1.27)
-				)
-			)
-		)
-		(property "Footprint" "Package_SO:TSSOP-28_4.4x9.7mm_P0.65mm"
-			(at 226.06 29.21 0)
-			(hide yes)
-			(show_name no)
-			(do_not_autoplace no)
-			(effects
-				(font
-					(size 1.27 1.27)
-				)
-			)
-		)
-		(property "Datasheet" ""
-			(at 226.06 29.21 0)
-			(hide yes)
-			(show_name no)
-			(do_not_autoplace no)
-			(effects
-				(font
-					(size 1.27 1.27)
-				)
-			)
-		)
-		(property "Description" "Special symbol for telling ERC where power comes from"
-			(at 226.06 29.21 0)
-			(hide yes)
-			(show_name no)
-			(do_not_autoplace no)
-			(effects
-				(font
-					(size 1.27 1.27)
-				)
-			)
-		)
-		(pin "1"
-		)
-		(instances
-			(project "mcu_datalogger"
-				(path "/c956c193-eb19-4c5d-8ea2-20354ad9de1d"
-					(reference "#FLG01")
-					(unit 1)
-				)
-			)
-		)
-	)
-	(symbol
 		(lib_id "Device:R")
 		(at 146.05 48.26 90)
@@
 		)
 		(pin "MOSI" input
-			(at 171.45 142.24 180)
+			(at 171.45 144.145 180)
 			(effects
 				(font
@@
 		)
 		(pin "RESET" passive
-			(at 171.45 147.32 180)
+			(at 171.45 149.225 180)
 			(effects
 				(font
@@
 		)
 		(pin "MISO" output
-			(at 171.45 144.78 180)
+			(at 171.45 146.685 180)
 			(effects
 				(font
@@
 			)
 		)
-		(pin "SCK" passive
+		(pin "SCL" passive
 			(at 171.45 132.08 180)
 			(effects
 				(font
+					(size 1.27 1.27)
+				)
+				(justify left)
+			)
+		)
+		(pin "SCK" passive
+			(at 171.45 141.605 180)
+			(effects
+				(font
