File: mcu_datalogger.kicad_pcb (KiCad board)
At the start: 2 copper layers, 38 x 47 mm, 29 parts, among them J1 Conn_01x04_Pin, J2 Conn_01x04_Pin, J3 Conn_01x09_Pin, J4 Conn_02x03_Odd_Even, U1 24LC1025, U2 DS1337S_, U3 24LC1025, U4 ATMEGA328P-AU_SL044, Y1 32.768 KHz, Y2 16 MHz

Commit message: optimisation
Parts:
- added G***: LOGO, _Logo:logo_2mm, B.Cu at (165.7, 91.4)
- moved J1 12.0 mm to (159.8, 64.7), turned to 90 degrees
- moved R4 6.73 mm to (156.6, 72.0)
- moved H1 4.30 mm to (170.7, 61.0)
- moved H4 4.30 mm to (170.7, 102.0)
- moved U1 3.99 mm to (166.7, 71.5)
- moved U3 3.99 mm to (160.7, 71.5)
- moved R6 1.28 mm to (154.3, 72.0)
- moved R3 1.08 mm to (152.0, 72.0)
Routing:
- net /SDA: track 63.1 -> 76.6 mm, vias 2 -> 4
- net GND: track 111.1 -> 102.3 mm, vias 2 -> 0
- net /Vcc: track 34.4 -> 39.9 mm
- net /SCL: track 58.7 -> 64.2 mm
- net /RESET: track 13.1 -> 11.8 mm
- net /SCK: track 37.0 -> 36.0 mm
Other:
- board size 38 x 47 mm -> 33.7 x 47 mm
- board text added: "SCL"
